Commit message: 可以运行setup_assistant的demo.launch.py

File: engineer_description/urdf/engineer_description.urdf (robot description, URDF)
Before this commit: robot engineer_description, 10 links, 9 joints
Joints:
- joint arm_pitch_joint: limit lower=0 upper=1.57 effort=100 velocity=1 -> lower=0 upper=1.57 effort=100 velocity=1.000001
- joint arm_roll_joint: limit lower=-6.28 upper=6.28 effort=100 velocity=1 -> lower=-6.28 upper=6.28 effort=100 velocity=1.000001
- joint arm_yaw_joint: limit lower=-0.5 upper=0.5 effort=100 velocity=1 -> lower=-0.5 upper=0.5 effort=100 velocity=1.000001
- joint extend_joint: limit lower=0 upper=0.66 effort=100 velocity=1 -> lower=0 upper=0.66 effort=100 velocity=1.000001
- joint pitch_joint: limit lower=-1.57 upper=1.57 effort=100 velocity=1 -> lower=-1.57 upper=1.57 effort=100 velocity=1.000001
- joint roll_joint: limit lower=-6.28 upper=6.28 effort=100 velocity=1 -> lower=-6.28 upper=6.28 effort=100 velocity=1.000001
- joint slide_joint: limit lower=0 upper=0.138 effort=100 velocity=1 -> lower=0 upper=0.138 effort=100 velocity=1.000001
- joint uplift_joint: limit lower=0 upper=0.66 effort=100 velocity=1 -> lower=0 upper=0.66 effort=100 velocity=1.000001

Commit message: moveit可以与gazebo联动

File: engineer_description/urdf/engineer_description.urdf (robot description, URDF)
Before this commit: robot engineer_description, 10 links, 9 joints
Links:
- link arm_pitch_Link: geometry collision mesh filename=file://$(find engineer_description)/meshes/arm_pitch_Link.S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; visual mesh filename=file://$(find engineer_description)/meshes/arm_pitch_Link.S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
- link arm_roll_Link: geometry collision mesh filename=file://$(find engineer_description)/meshes/arm_roll_Link.STL; visual mesh filename=file://$(find engineer_description)/meshes/arm_roll_Link.STL
- link arm_yaw_Link: geometry collision mesh filename=file://$(find engineer_description)/meshes/arm_yaw_Link.STL; visual mesh filename=file://$(find engineer_description)/meshes/arm_yaw_Link.STL
- link base_link: geometry collision mesh filename=file://$(find engineer_description)/meshes/base_link.STL; visual mesh filename=file://$(find engineer_description)/meshes/base_link.STL
- link extend_Link: geometry collision mesh filename=file://$(find engineer_description)/meshes/extend_Link.STL; visual mesh filename=file://$(find engineer_description)/meshes/extend_Link.STL
- link pitch_Link: geometry collision mesh filename=file://$(find engineer_description)/meshes/pitch_Link.STL; visual mesh filename=file://$(find engineer_description)/meshes/pitch_Link.STL
- link roll_Link: geometry collision mesh filename=file://$(find engineer_description)/meshes/roll_Link.STL; visual mesh filename=file://$(find engineer_description)/meshes/roll_Link.STL
- link slide_Link: geometry collision mesh filename=file://$(find engineer_description)/meshes/slide_Link.STL; visual mesh filename=file://$(find engineer_description)/meshes/slide_Link.STL
- link uplift_Link: geometry collision mesh filename=file://$(find engineer_description)/meshes/uplift_Link.STL; visual mesh filename=file://$(find engineer_description)/meshes/uplift_Link.STL
